Commit message: chlore: hauteur

File: description/Gazebo_control.xacro (robot description, xacro)
@@ -6,5 +6,5 @@
       <left_joint>left_wheel_joint</left_joint>
       <right_joint>right_wheel_joint</right_joint>
-      <wheel_separation>1.5</wheel_separation>
+      <wheel_separation>1.2</wheel_separation>
       <wheel_radius>0.4</wheel_radius>
       <topic>cmd_vel</topic>

File: description/building_robot.xacro (robot description, xacro)
@@ -24,5 +24,5 @@
   <link name="left_wheel">
     <inertial>
-      <mass value="1"/>
+      <mass value="0.5"/>
       <inertia ixx="0.043333" ixy="0" ixz="0" iyy="0.043333" iyz="0" izz="0.08"/>
     </inertial>
@@ -75,5 +75,5 @@
     <visual>
       <geometry>
-        <sphere radius="0.4"/>
+        <sphere radius="0.3"/>
       </geometry>
       <material name="green">

Commit message: Mise en place du mini robot avec les bonnes valeurs et les capteurs pour le physique dans gazebo

File: description/Gazebo_control.xacro (robot description, xacro)
@@ -6,8 +6,8 @@
       <left_joint>left_wheel_joint</left_joint>
       <right_joint>right_wheel_joint</right_joint>
-      <wheel_separation>1.2</wheel_separation>
-      <wheel_radius>0.4</wheel_radius>
+      <wheel_separation>2.2</wheel_separation>
+      <wheel_radius>0.5</wheel_radius>
       <topic>cmd_vel</topic>
-      <max_linear_acceleration>0.3</max_linear_acceleration>
+      <max_linear_acceleration>0.4</max_linear_acceleration>
       <frame_id>odom</frame_id>
       <child_frame_id>chassis</child_frame_id>

File: description/building_robot.xacro (robot description, xacro)
@@ -9,5 +9,5 @@
     <visual>
       <geometry>
-        <box size="2 1 0.5"/>
+        <box size="3 2 0.75"/>
       </geometry>
       <material name="blue">
@@ -17,5 +17,5 @@
     <collision>
       <geometry>
-        <box size="2 1 0.5"/>
+        <box size="3 2 0.75"/>
       </geometry>
     </collision>
@@ -29,5 +29,5 @@
     <visual>
       <geometry>
-        <cylinder radius="0.4" length="0.2"/>
+        <cylinder radius="0.5" length="0.2"/>
       </geometry>
       <material name="red">
@@ -37,5 +37,5 @@
     <collision>
       <geometry>
-        <cylinder radius="0.4" length="0.2"/>
+        <cylinder radius="0.5" length="0.2"/>
       </geometry>
       <material name="red">
@@ -52,5 +52,5 @@
     <visual>
       <geometry>
-        <cylinder radius="0.4" length="0.2"/>
+        <cylinder radius="0.5" length="0.2"/>
       </geometry>
       <material name="red">
@@ -60,5 +60,5 @@
     <collision>
       <geometry>
-        <cylinder radius="0.4" length="0.2"/>
+        <cylinder radius="0.5" length="0.2"/>
       </geometry>
       <material name="red">
@@ -75,5 +75,5 @@
     <visual>
       <geometry>
-        <sphere radius="0.3"/>
+        <sphere radius="0.2"/>
       </geometry>
       <material name="green">
@@ -91,5 +91,5 @@
     <parent link="chassis"/>
     <child link="left_wheel"/>
-    <origin xyz="0.8 0.7 -0.25" rpy="1.57 0 0"/>
+    <origin xyz="1.3 1.1 -0.20" rpy="1.57 0 0"/>
     <axis xyz="0 0 1"/>
   </joint>
@@ -97,5 +97,5 @@
     <parent link="chassis"/>
     <child link="right_wheel"/>
-    <origin xyz="0.8 -0.7 -0.25" rpy="-1.57 0 0"/>
+    <origin xyz="1.3 -1.1 -0.20" rpy="-1.57 0 0"/>
     <axis xyz="0 0 1"/>
   </joint>
@@ -103,5 +103,5 @@
     <parent link="chassis"/>
     <child link="caster"/>
-    <origin xyz="-0.8 0 -0.3" rpy="0 0 0"/>
+    <origin xyz="-1.3 0 -0.5" rpy="0 0 0"/>
   </joint>
 </robot>

File: description/camera.xacro (robot description, xacro)
@@ -4,17 +4,17 @@
         <parent link="chassis"/>
         <child link="camera_link"/>
-        <origin xyz="0.276 0 0.181" rpy="0 0 0"/>
+        <origin xyz="1.3 -0.75 0.6" rpy="0 0 0"/>
     </joint>
     <link name="camera_link">
         <visual>
             <geometry>
-                <box size="0.010 0.03 0.03"/>
+                <box size="0.050 0.050 0.5"/>
             </geometry>
             <material name="black"/>
         </visual>
         <visual>
-            <origin xyz="0 0 -0.05"/>
+            <origin xyz="0 0 0.25"/>
             <geometry>
-                <cylinder radius="0.002" length="0.1"/>
+                <cylinder radius="0.08" length="0.09"/>
             </geometry>
             <material name="black"/>

File: description/gps.xacro (robot description, xacro)
@@ -5,12 +5,11 @@
     <parent link="chassis"/>
     <child link="gnss_frame"/>
-    <!-- Positionne le GNSS (exemple au-dessus du châssis) -->
-    <origin xyz="0.10 0 0.80" rpy="0 0 0"/>
+    <origin xyz="1.3 0.75 0.60" rpy="0 0 0"/>
   </joint>
   <!-- Lien du capteur GNSS (petit cylindre pour le visuel) -->
   <link name="gnss_frame">
-   <visual>
+    <visual>
       <geometry>
-        <cylinder radius="0.03" length="0.02"/>
+        <cylinder radius="0.03" length="0.5"/>
       </geometry>
       <material name="black"/>
@@ -18,29 +17,24 @@
     <collision>
       <geometry>
-        <cylinder radius="0.03" length="0.02"/>
+        <cylinder radius="0.03" length="0.5"/>
       </geometry>
     </collision>
-    <xacro:inertial_cylinder mass="0.05" length="0.02" radius="0.03">
+    <xacro:inertial_cylinder mass="0.05" length="0.5" radius="0.03">
       <origin xyz="0 0 0" rpy="0 0 0"/>
     </xacro:inertial_cylinder>
   </link>
-  <!-- Définition du capteur GNSS pour Gazebo Sim -->
+  <!-- Capteur GNSS compatible Fortress -->
   <gazebo reference="gnss_frame">
-    <material>Gazebo/Black</material>
-    <!-- Capteur GNSS -->
-    <sensor name="gnss" type="navsat">
+    <sensor name="gnss_sensor" type="gps">
       <pose>0 0 0 0 0 0</pose>
-      <!-- topic côté Gazebo ; tu peux changer -->
-      <topic>/gnss/fix</topic>
-      <!-- Frame publiée (utile pour le bridge ROS2) -->
-      <gz_frame_id>gnss_frame</gz_frame_id>
       <update_rate>10</update_rate>
+      <topic>/gps/fix</topic>
+      <always_on>true</always_on>
       <navsat>
-        <!-- Modèle de bruit simple ; ajuste à ta convenance -->
         <position_sensing>
           <horizontal>
             <noise type="gaussian">
               <mean>0.0</mean>
-              <stddev>0.5</stddev>      <!-- ~0.5 m -->
+              <stddev>0.5</stddev>
             </noise>
           </horizontal>
@@ -48,5 +42,5 @@
             <noise type="gaussian">
               <mean>0.0</mean>
-              <stddev>1.0</stddev>      <!-- ~1.0 m -->
+              <stddev>1.0</stddev>
             </noise>
           </vertical>
@@ -55,9 +49,8 @@
           <noise type="gaussian">
             <mean>0.0</mean>
-            <stddev>0.1</stddev>        <!-- optionnel -->
+            <stddev>0.1</stddev>
           </noise>
         </velocity_sensing>
       </navsat>
-      <!-- Affichage dans l’UI de Gazebo (facultatif) -->
       <visualize>true</visualize>
     </sensor>

File: description/lidar.xacro (robot description, xacro)
@@ -5,17 +5,17 @@
         <parent link="chassis"/>
         <child link="laser_frame"/>
-        <origin xyz="0.122 0 0.212" rpy="0 0 0"/>
+        <origin xyz="-1.3 0 0.6" rpy="0 0 0"/>
     </joint>
     <link name="laser_frame">
         <visual>
             <geometry>
-                <cylinder radius="0.05" length="0.04"/>
+                <cylinder radius="0.3" length="0.09"/>
             </geometry>
             <material name="black"/>
         </visual>
         <visual>
-            <origin xyz="0 0 -0.05"/>
+            <origin xyz="0 0 -0.2"/>
             <geometry>
-                <cylinder radius="0.01" length="0.1"/>
+                <cylinder radius="0.175" length="0.5"/>
             </geometry>
             <material name="black"/>
@@ -23,41 +23,38 @@
         <collision>
             <geometry>
-                <cylinder radius="0.05" length="0.04"/>
+                <cylinder radius="0.3" length="0.09"/>
             </geometry>
         </collision>
-        <xacro:inertial_cylinder mass="0.1" length="0.04" radius="0.05">
+        <xacro:inertial_cylinder mass="0.1" length="0.09" radius="0.3">
             <origin xyz="0 0 0" rpy="0 0 0"/>
         </xacro:inertial_cylinder>
     </link>
-    <gazebo reference="laser_frame">
-        <material>Gazebo/Black</material>
-        <sensor name='laser' type='gpu_lidar'>
-            <pose>0 0 0 0 0 0</pose>
-            <topic>scan</topic>
-            <gz_frame_id>laser_frame</gz_frame_id>
-            <update_rate>10</update_rate>
-            <lidar>
-              <scan>
-                <horizontal>
-                  <samples>640</samples>
-                  <resolution>1</resolution>
-                  <min_angle>-1.396263</min_angle>
-                  <max_angle>1.396263</max_angle>
-                </horizontal>
-                <vertical>
-                  <samples>1</samples>
-                  <resolution>1</resolution>
-                  <min_angle>0.0</min_angle>
-                  <max_angle>0.0</max_angle>
-                </vertical>
-              </scan>
-              <range>
-                <min>0.08</min>
-                <max>10.0</max>
-                <resolution>0.01</resolution>
-              </range>
-            </lidar>
-            <visualize>true</visualize>
-          </sensor>
-    </gazebo>
+  <gazebo reference="laser_frame">
+    <sensor name="lidar_sensor" type="gpu_lidar">
+      <pose>0 0 0 0 0 0</pose>
+      <update_rate>10.0</update_rate>
+      <topic>/lidar/scan</topic>
+      <visualize>true</visualize>
+      <lidar>
+        <scan>
+          <horizontal>
+            <samples>640</samples>
+            <resolution>1</resolution>
+            <min_angle>-1.396263</min_angle>
+            <max_angle>1.396263</max_angle>
+          </horizontal>
+        </scan>
+        <range>
+          <min>0.08</min>
+          <max>10.0</max>
+          <resolution>0.01</resolution>
+        </range>
+      </lidar>
+      <noise>
+        <type>gaussian</type>
+        <mean>0.0</mean>
+        <stddev>0.01</stddev>
+      </noise>
+    </sensor>
+  </gazebo>
 </robot>
