Commit message: reconfiguration des capteurs

File: description/lidar.xacro (robot description, xacro)
@@ -5,5 +5,5 @@
         <parent link="chassis"/>
         <child link="laser_frame"/>
-        <origin xyz="-1.3 0 0.6" rpy="0 0 0"/>
+        <origin xyz="-1.3 0 0.5" rpy="0 0.2 3.1416"/>
     </joint>
     <link name="laser_frame">
@@ -34,5 +34,6 @@
       <pose>0 0 0 0 0 0</pose>
       <update_rate>10.0</update_rate>
-      <topic>/lidar/scan</topic>
+      <topic>/scan</topic>
+       <gz_frame_id>laser_frame</gz_frame_id>
       <visualize>true</visualize>
       <lidar>
@@ -44,4 +45,10 @@
             <max_angle>1.396263</max_angle>
           </horizontal>
+          <vertical>
+              <samples>1</samples>
+              <resolution>1</resolution>
+              <min_angle>0.0</min_angle>
+              <max_angle>0.0</max_angle>
+          </vertical>
         </scan>
         <range>
